Commit message: fixed integration and encoder

File: xacro/test.xacro (robot description, xacro)
@@ -68,4 +68,5 @@
     <xacro:property name="params_yaml" value="$(find gazebo_ros_motors)/params/dc_motor.yaml"/>
     <origin xyz="0 0 0.2" rpy="0 0 0"/>
+    <axis xyz="0 0 1" rpy="0 0 0"/> <!-- Without this an Not Enough Blocks error happens -->
   </xacro:dc_motor>
 </robot>
